Commit message: Interfaced Gazebo with ROS

File: Remote_System/remote_ws/src/sangi_description/urdf/sangi.xacro (robot description, xacro)
@@ -1,4 +1,4 @@
 <?xml version="1.0"?>
-<robot name="mybot" xmlns:xacro="http://www.ros.org/wiki/xacro">
+<robot name="sangi" xmlns:xacro="http://www.ros.org/wiki/xacro">
         <!-- Put here the robot description -->
 	<xacro:property name="PI" value="3.1415926535897931"/>
@@ -15,6 +15,57 @@
 	<xacro:property name="sonarSize" value="0.005"/>
 	<xacro:property name="sonarMass" value="0.01"/>
-	<xacro:include filename="$(find mybot_description)/urdf/mybot.gazebo" />
- 	<xacro:include filename="$(find mybot_description)/urdf/materials.xacro" />
- 	<xacro:include filename="$(find mybot_description)/urdf/macros.xacro" />
+	<xacro:include filename="$(find sangi_description)/urdf/sangi.gazebo" />
+ 	<xacro:include filename="$(find sangi_description)/urdf/materials.xacro" />
+ 	<xacro:include filename="$(find sangi_description)/urdf/macros.xacro" />
+	<link name="footprint" />
+	<joint name="base_joint" type="fixed">
+			<parent link="footprint"/>
+			<child link="chassis"/>
+	</joint>
+   <link name='chassis'>
+    <collision>
+      <origin xyz="0 0 ${wheelRadius}" rpy="0 0 0"/>
+      <geometry>
+        <box size="${chassisLength} ${chassisWidth} ${chassisHeight}"/>
+      </geometry>
+    </collision>
+    <visual>
+      <origin xyz="0 0 ${wheelRadius}" rpy="0 0 0"/>
+      <geometry>
+        <box size="${chassisLength} ${chassisWidth} ${chassisHeight}"/>
+      </geometry>
+      <material name="orange"/>
+    </visual>
+    <inertial>
+      <origin xyz="0 0 ${wheelRadius}" rpy="0 0 0"/>
+      <mass value="${chassisMass}"/>
+      <box_inertia m="${chassisMass}" x="${chassisLength}" y="${chassisWidth}" z="${chassisHeight}" />
+    </inertial>
+   </link>
+    <joint name="fixed" type="fixed">
+  <parent link="chassis"/>
+  <child link="caster_wheel"/>
+</joint>
+<link name="caster_wheel">
+  <collision>
+    <origin xyz="${casterRadius-chassisLength/2} 0 ${casterRadius-chassisHeight+wheelRadius}" rpy="0 0 0"/>
+    <geometry>
+      <sphere radius="${casterRadius}"/>
+    </geometry>
+  </collision>
+  <visual>
+    <origin xyz="${casterRadius-chassisLength/2} 0 ${casterRadius-chassisHeight+wheelRadius}" rpy="0 0 0"/>
+    <geometry>
+      <sphere radius="${casterRadius}"/>
+    </geometry>
+    <material name="red"/>
+  </visual>
+  <inertial>
+    <origin xyz="${casterRadius-chassisLength/2} 0 ${casterRadius-chassisHeight+wheelRadius}" rpy="0 0 0"/>
+    <mass value="${casterMass}"/>
+    <sphere_inertia m="${casterMass}" r="${casterRadius}"/>
+  </inertial>
+</link>
+<wheel lr="left" tY="1"/>
+<wheel lr="right" tY="-1"/>
 </robot>

Commit message: Simulation work

File: Remote_System/remote_ws/src/sangi_description/urdf/sangi.xacro (robot description, xacro)
@@ -67,5 +67,94 @@
   </inertial>
 </link>
-<wheel lr="left" tY="1"/>
-<wheel lr="right" tY="-1"/>
+<!-- <wheel lr="left" tY="1"/>
+<wheel lr="right" tY="-1"/> -->
+<!-- <link name="left_wheel">
+    <collision>
+      <origin xyz="0 0 0" rpy="0 ${PI/2} ${PI/2}" />
+      <geometry>
+        <cylinder length="${wheelWidth}" radius="${wheelRadius}"/>
+      </geometry>
+    </collision>
+    <visual>
+      <origin xyz="0 0 0" rpy="0 ${PI/2} ${PI/2}" />
+      <geometry>
+        <cylinder length="${wheelWidth}" radius="${wheelRadius}"/>
+      </geometry>
+      <material name="black"/>
+    </visual>
+    <inertial>
+      <origin xyz="0 0 0" rpy="0 ${PI/2} ${PI/2}" />
+      <mass value="${wheelMass}"/>
+      <cylinder_inertia m="${wheelMass}" r="${wheelRadius}" h="${wheelWidth}"/>
+    </inertial>
+  </link>
+  <gazebo reference="left_wheel">
+    <mu1 value="1.0"/>
+    <mu2 value="1.0"/>
+    <kp  value="10000000.0" />
+    <kd  value="1.0" />
+    <fdir1 value="1 0 0"/>
+    <material>Gazebo/Black</material>
+  </gazebo>
+  <joint name="left_wheel_hinge" type="continuous">
+    <parent link="chassis"/>
+    <child link="left_wheel"/>
+  <origin xyz="${-wheelPos+chassisLength/2} ${1*wheelWidth/2+1*chassisWidth/2} ${wheelRadius}" rpy="0 0 0" />
+    <axis xyz="0 1 0" rpy="0 0 0" />
+    <limit effort="100" velocity="100"/>
+    <joint_properties damping="0.0" friction="0.0"/>
+  </joint>
+  <transmission name="left_trans">
+    <type>transmission_interface/SimpleTransmission</type>
+    <joint name="left_wheel_hinge"/>
+    <actuator name="leftMotor">
+      <hardwareInterface>EffortJointInterface</hardwareInterface>
+      <mechanicalReduction>10</mechanicalReduction>
+    </actuator>
+  </transmission>
+<link name="right_wheel">
+    <collision>
+      <origin xyz="0 0 0" rpy="0 ${PI/2} ${PI/2}" />
+      <geometry>
+        <cylinder length="${wheelWidth}" radius="${wheelRadius}"/>
+      </geometry>
+    </collision>
+    <visual>
+      <origin xyz="0 0 0" rpy="0 ${PI/2} ${PI/2}" />
+      <geometry>
+        <cylinder length="${wheelWidth}" radius="${wheelRadius}"/>
+      </geometry>
+      <material name="black"/>
+    </visual>
+    <inertial>
+      <origin xyz="0 0 0" rpy="0 ${PI/2} ${PI/2}" />
+      <mass value="${wheelMass}"/>
+      <cylinder_inertia m="${wheelMass}" r="${wheelRadius}" h="${wheelWidth}"/>
+    </inertial>
+  </link>
+  <gazebo reference="right_wheel">
+    <mu1 value="1.0"/>
+    <mu2 value="1.0"/>
+    <kp  value="10000000.0" />
+    <kd  value="1.0" />
+    <fdir1 value="1 0 0"/>
+    <material>Gazebo/Black</material>
+  </gazebo>
+  <joint name="right_wheel_hinge" type="continuous">
+    <parent link="chassis"/>
+    <child link="right_wheel"/>
+  <origin xyz="${-wheelPos+chassisLength/2} ${-1*wheelWidth/2+-1*chassisWidth/2} ${wheelRadius}" rpy="0 0 0" />
+    <axis xyz="0 1 0" rpy="0 0 0" />
+    <limit effort="100" velocity="100"/>
+    <joint_properties damping="0.0" friction="0.0"/>
+  </joint>
+  <transmission name="right_trans">
+    <type>transmission_interface/SimpleTransmission</type>
+    <joint name="right_wheel_hinge"/>
+    <actuator name="rightMotor">
+      <hardwareInterface>EffortJointInterface</hardwareInterface>
+      <mechanicalReduction>10</mechanicalReduction>
+    </actuator>
+  </transmission>
+ -->
 </robot>

Commit message: Tf publishing properly

File: Remote_System/remote_ws/src/sangi_description/urdf/sangi.xacro (robot description, xacro)
@@ -67,94 +67,5 @@
   </inertial>
 </link>
-<!-- <wheel lr="left" tY="1"/>
-<wheel lr="right" tY="-1"/> -->
-<!-- <link name="left_wheel">
-    <collision>
-      <origin xyz="0 0 0" rpy="0 ${PI/2} ${PI/2}" />
-      <geometry>
-        <cylinder length="${wheelWidth}" radius="${wheelRadius}"/>
-      </geometry>
-    </collision>
-    <visual>
-      <origin xyz="0 0 0" rpy="0 ${PI/2} ${PI/2}" />
-      <geometry>
-        <cylinder length="${wheelWidth}" radius="${wheelRadius}"/>
-      </geometry>
-      <material name="black"/>
-    </visual>
-    <inertial>
-      <origin xyz="0 0 0" rpy="0 ${PI/2} ${PI/2}" />
-      <mass value="${wheelMass}"/>
-      <cylinder_inertia m="${wheelMass}" r="${wheelRadius}" h="${wheelWidth}"/>
-    </inertial>
-  </link>
-  <gazebo reference="left_wheel">
-    <mu1 value="1.0"/>
-    <mu2 value="1.0"/>
-    <kp  value="10000000.0" />
-    <kd  value="1.0" />
-    <fdir1 value="1 0 0"/>
-    <material>Gazebo/Black</material>
-  </gazebo>
-  <joint name="left_wheel_hinge" type="continuous">
-    <parent link="chassis"/>
-    <child link="left_wheel"/>
-  <origin xyz="${-wheelPos+chassisLength/2} ${1*wheelWidth/2+1*chassisWidth/2} ${wheelRadius}" rpy="0 0 0" />
-    <axis xyz="0 1 0" rpy="0 0 0" />
-    <limit effort="100" velocity="100"/>
-    <joint_properties damping="0.0" friction="0.0"/>
-  </joint>
-  <transmission name="left_trans">
-    <type>transmission_interface/SimpleTransmission</type>
-    <joint name="left_wheel_hinge"/>
-    <actuator name="leftMotor">
-      <hardwareInterface>EffortJointInterface</hardwareInterface>
-      <mechanicalReduction>10</mechanicalReduction>
-    </actuator>
-  </transmission>
-<link name="right_wheel">
-    <collision>
-      <origin xyz="0 0 0" rpy="0 ${PI/2} ${PI/2}" />
-      <geometry>
-        <cylinder length="${wheelWidth}" radius="${wheelRadius}"/>
-      </geometry>
-    </collision>
-    <visual>
-      <origin xyz="0 0 0" rpy="0 ${PI/2} ${PI/2}" />
-      <geometry>
-        <cylinder length="${wheelWidth}" radius="${wheelRadius}"/>
-      </geometry>
-      <material name="black"/>
-    </visual>
-    <inertial>
-      <origin xyz="0 0 0" rpy="0 ${PI/2} ${PI/2}" />
-      <mass value="${wheelMass}"/>
-      <cylinder_inertia m="${wheelMass}" r="${wheelRadius}" h="${wheelWidth}"/>
-    </inertial>
-  </link>
-  <gazebo reference="right_wheel">
-    <mu1 value="1.0"/>
-    <mu2 value="1.0"/>
-    <kp  value="10000000.0" />
-    <kd  value="1.0" />
-    <fdir1 value="1 0 0"/>
-    <material>Gazebo/Black</material>
-  </gazebo>
-  <joint name="right_wheel_hinge" type="continuous">
-    <parent link="chassis"/>
-    <child link="right_wheel"/>
-  <origin xyz="${-wheelPos+chassisLength/2} ${-1*wheelWidth/2+-1*chassisWidth/2} ${wheelRadius}" rpy="0 0 0" />
-    <axis xyz="0 1 0" rpy="0 0 0" />
-    <limit effort="100" velocity="100"/>
-    <joint_properties damping="0.0" friction="0.0"/>
-  </joint>
-  <transmission name="right_trans">
-    <type>transmission_interface/SimpleTransmission</type>
-    <joint name="right_wheel_hinge"/>
-    <actuator name="rightMotor">
-      <hardwareInterface>EffortJointInterface</hardwareInterface>
-      <mechanicalReduction>10</mechanicalReduction>
-    </actuator>
-  </transmission>
- -->
+<wheel lr="left" tY="1"/>
+<wheel lr="right" tY="-1"/>
 </robot>

Commit message: Added gas_station to the world

File: Remote_System/remote_ws/src/sangi_description/urdf/sangi.xacro (robot description, xacro)
@@ -43,8 +43,8 @@
     </inertial>
    </link>
-    <joint name="fixed" type="fixed">
-  <parent link="chassis"/>
-  <child link="caster_wheel"/>
-</joint>
+	<joint name="fixed" type="fixed">
+	  	<parent link="chassis"/>
+	  	<child link="caster_wheel"/>
+	</joint>
 <link name="caster_wheel">
   <collision>
@@ -69,3 +69,4 @@
 <wheel lr="left" tY="1"/>
 <wheel lr="right" tY="-1"/>
+<sonar name="sonar1" parent="chassis" origin="0 0 0" ros_topic="sonar1" update_rate="10" min_range="10" max_range="100" field_of_view="1" ray_count="10"/>
 </robot>
