Commit message: Worked on Simulation

File: Remote_System/remote_ws/src/sangi_description/urdf/macros.xacro (robot description, xacro)
@@ -58,5 +58,7 @@
   <transmission name="${lr}_trans">
     <type>transmission_interface/SimpleTransmission</type>
-    <joint name="${lr}_wheel_hinge"/>
+    <joint name="${lr}_wheel_hinge">
+      <hardwareInterface>EffortJointInterface</hardwareInterface>
+    </joint>
     <actuator name="${lr}Motor">
       <hardwareInterface>EffortJointInterface</hardwareInterface>

Commit message: Added Hector Sonar Macro

File: Remote_System/remote_ws/src/sangi_description/urdf/macros.xacro (robot description, xacro)
@@ -20,50 +20,111 @@
   </macro>
   <macro name="wheel" params="lr tY">
-  <link name="${lr}_wheel">
-    <collision>
-      <origin xyz="0 0 0" rpy="0 ${PI/2} ${PI/2}" />
-      <geometry>
-        <cylinder length="${wheelWidth}" radius="${wheelRadius}"/>
-      </geometry>
-    </collision>
-    <visual>
-      <origin xyz="0 0 0" rpy="0 ${PI/2} ${PI/2}" />
-      <geometry>
-        <cylinder length="${wheelWidth}" radius="${wheelRadius}"/>
-      </geometry>
-      <material name="black"/>
-    </visual>
-    <inertial>
-      <origin xyz="0 0 0" rpy="0 ${PI/2} ${PI/2}" />
-      <mass value="${wheelMass}"/>
-      <cylinder_inertia m="${wheelMass}" r="${wheelRadius}" h="${wheelWidth}"/>
-    </inertial>
-  </link>
-  <gazebo reference="${lr}_wheel">
-    <mu1 value="100.0"/>
-    <mu2 value="100.0"/>
-    <kp  value="10000000.0" />
-    <kd  value="1.0" />
-    <fdir1 value="1 0 0"/>
-    <material>Gazebo/Black</material>
-  </gazebo>
-  <joint name="${lr}_wheel_hinge" type="continuous">
-    <parent link="chassis"/>
-    <child link="${lr}_wheel"/>
-  <origin xyz="${-wheelPos+chassisLength/2} ${tY*wheelWidth/2+tY*chassisWidth/2} ${wheelRadius}" rpy="0 0 0" />
-    <axis xyz="0 1 0" rpy="0 0 0" />
-    <limit effort="100" velocity="100"/>
-    <joint_properties damping="0.0" friction="0.0"/>
-  </joint>
-  <transmission name="${lr}_trans">
-    <type>transmission_interface/SimpleTransmission</type>
-    <joint name="${lr}_wheel_hinge">
-      <hardwareInterface>EffortJointInterface</hardwareInterface>
+	  <link name="${lr}_wheel">
+	    <collision>
+	      <origin xyz="0 0 0" rpy="0 ${PI/2} ${PI/2}" />
+	      <geometry>
+		<cylinder length="${wheelWidth}" radius="${wheelRadius}"/>
+	      </geometry>
+	    </collision>
+	    <visual>
+	      <origin xyz="0 0 0" rpy="0 ${PI/2} ${PI/2}" />
+	      <geometry>
+		<cylinder length="${wheelWidth}" radius="${wheelRadius}"/>
+	      </geometry>
+	      <material name="black"/>
+	    </visual>
+	    <inertial>
+	      <origin xyz="0 0 0" rpy="0 ${PI/2} ${PI/2}" />
+	      <mass value="${wheelMass}"/>
+	      <cylinder_inertia m="${wheelMass}" r="${wheelRadius}" h="${wheelWidth}"/>
+	    </inertial>
+	  </link>
+	  <gazebo reference="${lr}_wheel">
+	    <mu1 value="100.0"/>
+	    <mu2 value="100.0"/>
+	    <kp  value="10000000.0" />
+	    <kd  value="1.0" />
+	    <fdir1 value="1 0 0"/>
+	    <material>Gazebo/Black</material>
+	  </gazebo>
+	  <joint name="${lr}_wheel_hinge" type="continuous">
+	    <parent link="chassis"/>
+	    <child link="${lr}_wheel"/>
+	  <origin xyz="${-wheelPos+chassisLength/2} ${tY*wheelWidth/2+tY*chassisWidth/2} ${wheelRadius}" rpy="0 0 0" />
+	    <axis xyz="0 1 0" rpy="0 0 0" />
+	    <limit effort="100" velocity="100"/>
+	    <joint_properties damping="0.0" friction="0.0"/>
+	  </joint>
+	  <transmission name="${lr}_trans">
+	    <type>transmission_interface/SimpleTransmission</type>
+	    <joint name="${lr}_wheel_hinge">
+	      <hardwareInterface>EffortJointInterface</hardwareInterface>
+	    </joint>
+	    <actuator name="${lr}Motor">
+	      <hardwareInterface>EffortJointInterface</hardwareInterface>
+	      <mechanicalReduction>10</mechanicalReduction>
+	    </actuator>
+	  </transmission>
+  </macro>
+  <macro name="sonar_sensor" params="name parent *origin ros_topic update_rate min_range max_range field_of_view ray_count">
+    <joint name="${name}_joint" type="fixed">
+      <xacro:insert_block name="origin" />
+      <parent link="${parent}"/>
+      <child link="${name}_link"/>
     </joint>
-    <actuator name="${lr}Motor">
-      <hardwareInterface>EffortJointInterface</hardwareInterface>
-      <mechanicalReduction>10</mechanicalReduction>
-    </actuator>
-  </transmission>
-</macro>
+    <link name="${name}_link">
+      <inertial>
+        <mass value="0.001" />
+        <origin xyz="0 0 0" rpy="0 0 0" />
+        <inertia ixx="0.000000017" ixy="0" ixz="0" iyy="0.000000017" iyz="0" izz="0.000000017" />
+      </inertial>
+      <visual>
+        <origin xyz="0 0 0" rpy="0 0 0" />
+        <geometry>
+          <!--<box size="0.01 0.01 0.01" /> -->
+          <mesh filename="package://hector_sensors_description/meshes/sonar_sensor/max_sonar_ez4.dae"/>
+        </geometry>
+      </visual>
+      <collision>
+        <origin xyz="0 0 0" rpy="0 0 0" />
+        <geometry>
+          <box size="0.01 0.01 0.01" />
+        </geometry>
+      </collision>
+    </link>
+    <gazebo reference="${name}_link">
+      <sensor type="ray" name="${name}">
+        <always_on>true</always_on>
+        <update_rate>${update_rate}</update_rate>
+        <pose>0 0 0 0 0 0</pose>
+        <visualize>false</visualize>
+        <ray>
+          <scan>
+            <horizontal>
+              <samples>${ray_count}</samples>
+              <resolution>1</resolution>
+              <min_angle>-${field_of_view/2}</min_angle>
+              <max_angle> ${field_of_view/2}</max_angle>
+            </horizontal>
+            <vertical>
+              <samples>${ray_count}</samples>
+              <resolution>1</resolution>
+              <min_angle>-${field_of_view/2}</min_angle>
+              <max_angle> ${field_of_view/2}</max_angle>
+            </vertical>
+          </scan>
+          <range>
+            <min>${min_range}</min>
+            <max>${max_range}</max>
+            <resolution>0.01</resolution>
+          </range>
+        </ray>
+        <plugin name="gazebo_ros_${name}_controller" filename="libhector_gazebo_ros_sonar.so">
+          <gaussianNoise>0.005</gaussianNoise>
+          <topicName>${ros_topic}</topicName>
+          <frameId>${name}_link</frameId>
+        </plugin>
+      </sensor>
+    </gazebo>
+  </macro>
 </robot>

Commit message: Added 3 sonars

File: Remote_System/remote_ws/src/sangi_description/urdf/macros.xacro (robot description, xacro)
@@ -67,7 +67,7 @@
 	  </transmission>
   </macro>
-  <macro name="sonar_sensor" params="name parent *origin ros_topic update_rate min_range max_range field_of_view ray_count">
+    <xacro:macro name="sonar_sensor" params="name parent ros_topic origin_new update_rate min_range max_range field_of_view ray_count">
     <joint name="${name}_joint" type="fixed">
-      <xacro:insert_block name="origin" />
+      <!--<xacro:insert_block name="origin" />!-->
       <parent link="${parent}"/>
       <child link="${name}_link"/>
@@ -76,9 +76,9 @@
       <inertial>
         <mass value="0.001" />
-        <origin xyz="0 0 0" rpy="0 0 0" />
+        <origin xyz="${origin_new}" rpy="0 0 0" />
         <inertia ixx="0.000000017" ixy="0" ixz="0" iyy="0.000000017" iyz="0" izz="0.000000017" />
       </inertial>
       <visual>
-        <origin xyz="0 0 0" rpy="0 0 0" />
+        <origin xyz="${origin_new}" rpy="0 0 0" />
         <geometry>
           <!--<box size="0.01 0.01 0.01" /> -->
@@ -87,7 +87,7 @@
       </visual>
       <collision>
-        <origin xyz="0 0 0" rpy="0 0 0" />
+        <origin xyz="${origin_new}" rpy="0 0 0" />
         <geometry>
-          <box size="0.01 0.01 0.01" />
+          <box size="0.05 0.05 0.05" />
         </geometry>
       </collision>
@@ -127,4 +127,4 @@
       </sensor>
     </gazebo>
-  </macro>
+  </xacro:macro>
 </robot>

File: Remote_System/remote_ws/src/sangi_description/urdf/sangi.xacro (robot description, xacro)
@@ -69,4 +69,6 @@
 <wheel lr="left" tY="1"/>
 <wheel lr="right" tY="-1"/>
-<sonar name="sonar1" parent="chassis" origin="0 0 0" ros_topic="sonar1" update_rate="10" min_range="10" max_range="100" field_of_view="1" ray_count="10"/>
+<sonar_sensor name="sonar1" parent="chassis" ros_topic="sonar1" origin_new="${chassisLength/2} 0 ${chassisHeight}" update_rate="10" min_range="1" max_range="10" field_of_view="3.14" ray_count="1"/>
+<sonar_sensor name="sonar2" parent="chassis" ros_topic="sonar2" origin_new="${chassisLength/2} ${chassisWidth/2} ${chassisHeight}" update_rate="10" min_range="1" max_range="10" field_of_view="3.14" ray_count="1"/>
+<sonar_sensor name="sonar3" parent="chassis" ros_topic="sonar3" origin_new="${chassisLength/2} -${chassisWidth/2} ${chassisHeight}" update_rate="10" min_range="1" max_range="10" field_of_view="3.14" ray_count="1"/>
 </robot>

Commit message: #6 Added indoor world and changed sonar positioning

File: Remote_System/remote_ws/src/sangi_description/urdf/macros.xacro (robot description, xacro)
@@ -67,5 +67,5 @@
 	  </transmission>
   </macro>
-    <xacro:macro name="sonar_sensor" params="name parent ros_topic origin_new update_rate min_range max_range field_of_view ray_count">
+    <xacro:macro name="sonar_sensor" params="name parent ros_topic origin_new rpy update_rate min_range max_range field_of_view ray_count">
     <joint name="${name}_joint" type="fixed">
       <!--<xacro:insert_block name="origin" />!-->
@@ -76,9 +76,9 @@
       <inertial>
         <mass value="0.001" />
-        <origin xyz="${origin_new}" rpy="0 0 0" />
+        <origin xyz="${origin_new}" rpy="${rpy}" />
         <inertia ixx="0.000000017" ixy="0" ixz="0" iyy="0.000000017" iyz="0" izz="0.000000017" />
       </inertial>
       <visual>
-        <origin xyz="${origin_new}" rpy="0 0 0" />
+        <origin xyz="${origin_new}" rpy="${rpy}" />
         <geometry>
           <!--<box size="0.01 0.01 0.01" /> -->
@@ -87,5 +87,5 @@
       </visual>
       <collision>
-        <origin xyz="${origin_new}" rpy="0 0 0" />
+        <origin xyz="${origin_new}" rpy="${rpy}" />
         <geometry>
           <box size="0.05 0.05 0.05" />

File: Remote_System/remote_ws/src/sangi_description/urdf/sangi.xacro (robot description, xacro)
@@ -69,6 +69,6 @@
 <wheel lr="left" tY="1"/>
 <wheel lr="right" tY="-1"/>
-<sonar_sensor name="sonar1" parent="chassis" ros_topic="sonar1" origin_new="${chassisLength/2} 0 ${chassisHeight}" update_rate="10" min_range="1" max_range="10" field_of_view="3.14" ray_count="1"/>
-<sonar_sensor name="sonar2" parent="chassis" ros_topic="sonar2" origin_new="${chassisLength/2} ${chassisWidth/2} ${chassisHeight}" update_rate="10" min_range="1" max_range="10" field_of_view="3.14" ray_count="1"/>
-<sonar_sensor name="sonar3" parent="chassis" ros_topic="sonar3" origin_new="${chassisLength/2} -${chassisWidth/2} ${chassisHeight}" update_rate="10" min_range="1" max_range="10" field_of_view="3.14" ray_count="1"/>
+<sonar_sensor name="sonar1" parent="chassis" ros_topic="sonar1" origin_new="${chassisLength/2} 0 ${chassisHeight}" rpy="0 0 0" update_rate="10" min_range="1" max_range="10" field_of_view="3.14" ray_count="1"/>
+<sonar_sensor name="sonar2" parent="chassis" ros_topic="sonar2" origin_new="${chassisLength/2} ${chassisWidth/2} ${chassisHeight}" rpy="0 0 1.57" update_rate="10" min_range="1" max_range="10" field_of_view="3.14" ray_count="1"/>
+<sonar_sensor name="sonar3" parent="chassis" ros_topic="sonar3" origin_new="${chassisLength/2} -${chassisWidth/2} ${chassisHeight}" rpy="0 0 -1.57" update_rate="10" min_range="1" max_range="10" field_of_view="3.14" ray_count="1"/>
 </robot>

Commit message: Added control for sonar mesh and hector plugins to prevent external download

File: Remote_System/remote_ws/src/sangi_description/urdf/macros.xacro (robot description, xacro)
@@ -83,5 +83,5 @@
         <geometry>
           <!--<box size="0.01 0.01 0.01" /> -->
-          <mesh filename="package://hector_sensors_description/meshes/sonar_sensor/max_sonar_ez4.dae"/>
+          <mesh filename="package://sangi_description/meshes/sonar/ping_sonar.dae"/>
         </geometry>
       </visual>
